File: hardware/interface-osi/addon.kicad_sch (KiCad schematic)
At the start: 22 parts, among them J1 Conn_01x16, U1 4066, U2 74HC14

Commit message: Cleanup RESET+SHIFTLOCK addon
- replaced DIP header with 13-pin 0.1" vertical header.  Added labels to
the pins.

- removed left over unused diode

- reversed default on / default off labels on shiftlock mode jumper
block.
Parts:
- removed J1: Conn_01x16, Package_DIP:DIP-16_W7.62mm_Socket, symbol Connector_Generic:Conn_01x16
- added J1: Conn_01x13_Male, Connector_PinHeader_2.54mm:PinHeader_1x13_P2.54mm_Vertical, symbol Connector:Conn_01x13_Male
Connections:
- net +5V: now also J1.1 (Pin_1), J1.13 (Pin_13), J1.8 (Pin_8)
- net Break1: now also J1.3 (Pin_3)
- net Col0: now also J1.10 (Pin_10)
- net GND: now also J1.12 (Pin_12), J1.2 (Pin_2), J1.4 (Pin_4), J1.7 (Pin_7)
- net Row0: now also J1.11 (Pin_11)
- net ShiftLock1: now also J1.6 (Pin_6)
- net ShiftLockLED-: now also J1.9 (Pin_9)
- net ~{RESET}: now also J1.5 (Pin_5)
- no-connect marks 4 -> 0
Other:
- company: (none) -> OSIWeb.org
- title: OSI ~RESET~ and SHIFTLOCK circuits -> RESET and SHIFTLOCK circuits
