File: hardware/interface-osi/addon.kicad_pcb (KiCad board)
At the start: 2 copper layers, 43.2 x 60.5 mm, 26 parts, among them J1 Conn_01x13_Male, U1 4066, U2 74HC14

Commit message: More Interface-ASCII PCB cleanups
Changed lines of the file:
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@@
     (title "RESET and SHIFT LOCK")
     (date "2022-04-07")
-    (rev "1.4")
+    (rev "2")
     (company "OSIWeb.org")
   )
@@
       (effects (font (size 1 1) (thickness 0.15)))
     )
-    (fp_text value "1k" (at 5.08 2.37) (layer "F.Fab")
+    (fp_text value "1k" (at 2.6543 2.032) (layer "F.Fab")
       (effects (font (size 1 1) (thickness 0.15)))
     )
@@
       (effects (font (size 1 1) (thickness 0.15)))
     )
-    (fp_text value "4066" (at 3.81 17.57) (layer "F.Fab")
-      (effects (font (size 1 1) (thickness 0.15)))
+    (fp_text value "4066" (at 5.6134 17.2212) (layer "F.Fab")
+      (effects (font (size 0.635 0.635) (thickness 0.127)))
     )
     (fp_text user "${REFERENCE}" (at 3.81 7.62) (layer "F.Fab")
@@
       (effects (font (size 1 1) (thickness 0.15)))
     )
-    (fp_text value "0.1uF" (at 1.25 3.5) (layer "F.Fab")
+    (fp_text value "0.1uF" (at 2.4511 0.3429) (layer "F.Fab")
       (effects (font (size 1 1) (thickness 0.15)))
     )
@@
       (effects (font (size 1 1) (thickness 0.15)))
     )
-    (fp_text value "74HC14" (at 3.81 17.57) (layer "F.Fab")
-      (effects (font (size 1 1) (thickness 0.15)))
+    (fp_text value "74HC14" (at 3.6322 17.2212) (layer "F.Fab")
+      (effects (font (size 0.635 0.635) (thickness 0.127)))
     )
     (fp_text user "${REFERENCE}" (at 3.81 7.62) (layer "F.Fab")
@@
     (effects (font (size 0.635 0.635) (thickness 0.127)))
   )
-  (gr_text "${COMPANY} 2022" (at 120.142 97.282) (layer "F.SilkS")
+  (gr_text "${COMPANY} 2022" (at 120.65 97.2312) (layer "F.SilkS")
     (effects (font (size 1.016 1.016) (thickness 0.1524)))
   )
