File: hardware/interface-ascii/interface-ascii.kicad_pcb (KiCad board)
At the start: 2 copper layers, 88.9 x 132.1 mm, 48 parts, among them J1 Apple 2, J2 Apple 1, J3 UART, J4 Outputs, J5 ISP header, J6 Keyboard, J7 SOL-20, SW1 Options, U1 ATmega328P, U2 74LS166, U3 74LS138, U4 74LS138, U5 74LS04

Commit message: production cleanup for interface-ascii
- Add production package scripts
- Configure BOM generation for KiBOM
- Add 3D models to path (add kicad 5 path variable to list)
- bump version to 3 for compatibility with versioning scheme
Connections:
- net /~RESET renamed /~{RESET}
- net /~STROBE renamed /~{STROBE}
Other:
- net class Default removed
- net class power1 removed
- net class signal removed
- board text added: "O3/~{RESET}"
- board text added: "OSIWeb.org 2019-22"
- board text added: "Unified Keyboard ASCII Interface Rev ${REVISION}"
- board text removed: "O3/~RESET"
- board text removed: "OSIWeb.org 2019-21"
- board text removed: "Unified Keyboard ASCII Interface Rev 2.11"

Commit message: More Interface-ASCII PCB cleanups
Parts:
- removed ?: , 
- added R1: 470, Resistor_THT:R_Axial_DIN0207_L6.3mm_D2.5mm_P10.16mm_Horizontal, F.Cu at (230.5, 65.2)
Connections:
- J1 pad 14: Net-(J1-Pad14) -> unconnected-(J1-Pad14)
- J1 pad 15: Net-(J1-Pad15) -> unconnected-(J1-Pad15)
- J1 pad 16: Net-(J1-Pad16) -> unconnected-(J1-Pad16)
- J1 pad 4: Net-(J1-Pad4) -> unconnected-(J1-Pad4)
- J1 pad 9: Net-(J1-Pad9) -> unconnected-(J1-Pad9)
- J2 pad 10: Net-(J2-Pad10) -> unconnected-(J2-Pad10)
- J2 pad 11: Net-(J2-Pad11) -> unconnected-(J2-Pad11)
- J2 pad 13: Net-(J2-Pad13) -> unconnected-(J2-Pad13)
- J3 pad 2: /D1 -> /Tx
- J6 pad 26: Net-(J6-Pad26) -> unconnected-(J6-Pad26)
- J6 pad 28: Net-(J6-Pad28) -> unconnected-(J6-Pad28)
- J6 pad 30: Net-(J6-Pad30) -> unconnected-(J6-Pad30)
- J6 pad 32: Net-(J6-Pad32) -> unconnected-(J6-Pad32)
- U2 pad 9: Net-(U2-Pad9) -> +5V
- U5 pad 10: Net-(U5-Pad10) -> unconnected-(U5-Pad10)
- U5 pad 6: Net-(U5-Pad6) -> unconnected-(U5-Pad6)
- U5 pad 8: Net-(U5-Pad8) -> unconnected-(U5-Pad8)
Routing:
- net +5V: track 557.0 -> 517.2 mm, vias 7 -> 8
- net /D1: track 134.6 -> 117.1 mm
- net /Tx: track 0.00 -> 7.11 mm
- net GND: track 481.5 -> 480.3 mm
- net Net-(D17-Pad1): track 37.6 -> 36.7 mm
- net /Col7: track 60.0 -> 59.1 mm
- net /SCK-LED2: track 90.1 -> 89.2 mm
- net Net-(D6-Pad1): track 18.9 -> 18.4 mm
- net /Row0: track 56.0 -> 55.5 mm
- net (no net): vias 1 -> 0
