File: hardware/keyboard-classic/kbd-classic.kicad_pcb (KiCad board)
At the start: 2 copper layers, 346.1 x 116.8 mm, 143 parts, among them J1 Controller, SW1 RT Arrow, SW10 Bracket_Open, SW11 6, SW12 Y, SW13 Return, SW14 Dash, SW15 5, SW16 T, SW17 Line_Feed, SW18 Colon, SW19 4, SW2 LT Arrow, SW20 R, SW21 O, SW22 0, SW23 3, SW24 E, SW25 L, SW26 9, SW27 2, SW28 W, SW29 Period, SW3 Tilde, SW30 8, SW31 1, SW32 @(OSI SL), SW33 Break, SW34 Rubout (OSI Break), SW35 R_Shift, SW36 P, SW37 Comma, SW38 K, SW39 L_Shift, SW4 I, SW40 Semicolon, SW41 M, SW42 J, SW43 Fwd_Slash, SW44 N, SW45 H, SW46 SPACE, SW47 B, SW48 G, SW49 TAB, SW5 Repeat, SW50 Z, SW51 V, SW52 F, SW53 CTRL, SW54 A, SW55 C, SW56 D, SW57 Backslash, SW58 Q, SW59 X, SW6 Bracket_Close, SW60 S, SW61 Power Light, SW62 ESC, SW63 Spare, SW7 7, SW8 U, SW9 Caps_Lock

Commit message: Update classic keyboard main PCB to kicad 6
- fix various ERC and DRC errors resulting from upgrade

- list included nets in busses on schematic

- Modify Footprints with multiple options (therefore multiple sets of
pads) to used shaped pads and proper pad numbering to eliminate DRC
issues, and ensure proper behavior
Parts:
- removed REF**: OSI mounting holes, unikbd:OSI mounting holes
- removed REF** (x7): MountingHole_3.5mm, MountingHole:MountingHole_3.5mm
Connections:
- J1 pad 26: Net-(J1-Pad26) -> unconnected-(J1-Pad26)
- J1 pad 28: Net-(J1-Pad28) -> unconnected-(J1-Pad28)
- J1 pad 30: Net-(J1-Pad30) -> unconnected-(J1-Pad30)
- J1 pad 32: Net-(J1-Pad32) -> unconnected-(J1-Pad32)
- J1 pad 33: Net-(J1-Pad33) -> unconnected-(J1-Pad33)
- J1 pad 34: Net-(J1-Pad34) -> unconnected-(J1-Pad34)
- J1 pad 35: Net-(J1-Pad35) -> unconnected-(J1-Pad35)
- J1 pad 36: Net-(J1-Pad36) -> unconnected-(J1-Pad36)
- J1 pad 37: Net-(J1-Pad37) -> unconnected-(J1-Pad37)
- J1 pad 38: Net-(J1-Pad38) -> unconnected-(J1-Pad38)
- J1 pad 39: Net-(J1-Pad39) -> unconnected-(J1-Pad39)
- J1 pad 40: Net-(J1-Pad40) -> unconnected-(J1-Pad40)
Routing:
- net Net-(D33-Pad2): track 195.2 -> 187.5 mm, vias 1 -> 0
- net Net-(D47-Pad2): track 17.1 -> 10.4 mm
- net /Row3: track 341.4 -> 340.0 mm
- net /Row2: track 319.3 -> 318.1 mm
- net Net-(D63-Pad1): track 193.4 -> 192.6 mm
- net /Col4: track 414.5 -> 413.8 mm
- net Net-(D63-Pad2): track 100.5 -> 99.8 mm
- net /Col7: track 389.8 -> 389.2 mm
- net Net-(J1-Pad2): track 239.1 -> 238.6 mm
- net /Col0: track 156.3 -> 155.8 mm
- net /Col2: track 501.4 -> 501.2 mm, vias 8 -> 7
Other:
- net class Default removed
- net class power1 removed
- net class signal removed

Commit message: Restore mounting holes
A prior commit apparently deleted several mounting holes.

- restore mounting holes
- update to Kicad7
- fix DRC errors resulting from update
- update footprints to use new shaped pads
Parts:
- added REF**: MountingHole_3.5mm, MountingHole:MountingHole_3.5mm, F.Cu at (67.3, 77.5)
- added REF**: MountingHole_3.5mm, MountingHole:MountingHole_3.5mm, F.Cu at (67.3, 171.4)
- added REF**: OSI mounting holes, unikbd:OSI mounting holes, F.Cu at (197.2, 166.0)
- added REF**: MountingHole_3.5mm, MountingHole:MountingHole_3.5mm, F.Cu at (143.5, 77.5)
- added REF**: MountingHole_3.5mm, MountingHole:MountingHole_3.5mm, F.Cu at (290.8, 77.5)
- added REF**: MountingHole_3.5mm, MountingHole:MountingHole_3.5mm, F.Cu at (102.7, 171.4)
- added REF**: MountingHole_3.5mm, MountingHole:MountingHole_3.5mm, F.Cu at (217.2, 77.5)
- added REF**: MountingHole_3.5mm, MountingHole:MountingHole_3.5mm, F.Cu at (364.5, 77.5)
Connections:
- J1 pad 26: unconnected-(J1-Pad26) -> Net-(J1-Pad26)
- J1 pad 28: unconnected-(J1-Pad28) -> Net-(J1-Pad28)
- J1 pad 30: unconnected-(J1-Pad30) -> Net-(J1-Pad30)
- J1 pad 32: unconnected-(J1-Pad32) -> Net-(J1-Pad32)
- J1 pad 33: unconnected-(J1-Pad33) -> Net-(J1-Pad33)
- J1 pad 34: unconnected-(J1-Pad34) -> Net-(J1-Pad34)
- J1 pad 35: unconnected-(J1-Pad35) -> Net-(J1-Pad35)
- J1 pad 36: unconnected-(J1-Pad36) -> Net-(J1-Pad36)
- J1 pad 37: unconnected-(J1-Pad37) -> Net-(J1-Pad37)
- J1 pad 38: unconnected-(J1-Pad38) -> Net-(J1-Pad38)
- J1 pad 39: unconnected-(J1-Pad39) -> Net-(J1-Pad39)
- J1 pad 40: unconnected-(J1-Pad40) -> Net-(J1-Pad40)
