File: hardware/keyboard-classic/kbd-classic.kicad_pcb (KiCad board)
At the start: 2 copper layers, 346.1 x 116.8 mm, 143 parts, among them J1 Controller, SW1 RT Arrow, SW10 Bracket_Open, SW11 6, SW12 Y, SW13 Return, SW14 Dash, SW15 5, SW16 T, SW17 Line_Feed, SW18 Colon, SW19 4, SW2 LT Arrow, SW20 R, SW21 O, SW22 0, SW23 3, SW24 E, SW25 L, SW26 9, SW27 2, SW28 W, SW29 Period, SW3 Tilde, SW30 8, SW31 1, SW32 @(OSI SL), SW33 Break, SW34 Rubout (OSI Break), SW35 R_Shift, SW36 P, SW37 Comma, SW38 K, SW39 L_Shift, SW4 I, SW40 Semicolon, SW41 M, SW42 J, SW43 Fwd_Slash, SW44 N, SW45 H, SW46 SPACE, SW47 B, SW48 G, SW49 TAB, SW5 Repeat, SW50 Z, SW51 V, SW52 F, SW53 CTRL, SW54 A, SW55 C, SW56 D, SW57 Backslash, SW58 Q, SW59 X, SW6 Bracket_Close, SW60 S, SW61 Power Light, SW62 ESC, SW63 Spare, SW7 7, SW8 U, SW9 Caps_Lock

Commit message: Update to include mounting hardware
- Fix all components to include full information including BOM
information

- Include all mounting hardware in components List

- fix schematic to align on 0.1" grid.
Parts:
- renumbered D62 to LED1, D63 to LED2, D64 to LED3, D33 to LED4, D65 to LED5
Connections:
- J1 pad 26: Net-(J1-Pad26) -> unconnected-(J1-Pin_26-Pad26)
- J1 pad 28: Net-(J1-Pad28) -> unconnected-(J1-Pin_28-Pad28)
- J1 pad 30: Net-(J1-Pad30) -> unconnected-(J1-Pin_30-Pad30)
- J1 pad 32: Net-(J1-Pad32) -> unconnected-(J1-Pin_32-Pad32)
- J1 pad 33: Net-(J1-Pad33) -> unconnected-(J1-Pin_33-Pad33)
- J1 pad 34: Net-(J1-Pad34) -> unconnected-(J1-Pin_34-Pad34)
- J1 pad 35: Net-(J1-Pad35) -> unconnected-(J1-Pin_35-Pad35)
- J1 pad 36: Net-(J1-Pad36) -> unconnected-(J1-Pin_36-Pad36)
- J1 pad 37: Net-(J1-Pad37) -> unconnected-(J1-Pin_37-Pad37)
- J1 pad 38: Net-(J1-Pad38) -> unconnected-(J1-Pin_38-Pad38)
- J1 pad 39: Net-(J1-Pad39) -> unconnected-(J1-Pin_39-Pad39)
- J1 pad 40: Net-(J1-Pad40) -> unconnected-(J1-Pin_40-Pad40)
