File: hardware/keyboard-sol/kbd-sol.kicad_pcb (KiCad board)
At the start: 2 copper layers, 396.2 x 117.7 mm, 192 parts, among them J1 Controller, SW10 TAB: 1.25x, SW11 I, SW12 2, SW13 Zero, SW14 Q, SW15 O, SW16 3, SW17 Dash, SW18 W, SW19 P, SW20 4, SW21 Caret, SW22 E, SW23 AT, SW24 5, SW25 LT Bracket, SW26 R, SW27 Return: 1.5x, SW28 6, SW29 Backslash, SW30 T, SW31 Line Feed, SW32 7, SW33 RT Bracket, SW34 Y, SW35 Load, SW36 LT Ctrl, SW37 J, SW38 Upper Case: 1.5x, SW39 M, SW4 ESC: 1.75x, SW40 Shift Lock: 1.5x, SW41 K, SW42 LT Shift: 1.5x, SW43 Comma, SW44 A, SW45 L, SW46 Z, SW47 Period, SW48 S, SW49 Semicolon, SW5 8, SW50 X, SW51 Slash, SW52 D, SW53 Colon, SW54 C, SW55 RT Shift: 2x, SW56 F, SW57 DEL, SW58 V, SW59 Mode Select: 1.75x, SW6 BREAK, SW60 G, SW61 Repeat: 1.25x, SW62 B, SW63 H, SW64 RT Ctrl, SW65 N, SW66 Local, SW67 NP Dash, SW68 NP 4, SW69 NP Zero, SW7 U, SW70 Up Arrow, SW71 NP 7, SW72 NP 1, SW73 NP period, SW74 LT Arrow, SW75 NP asterisk, SW76 NP 5, SW77 NP plus, SW78 Spacebar, SW79 NP 8, SW8 1, SW80 NP 2, SW81 RT Arrow, SW82 NP divide, SW83 NP 6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

Commit message: Update the keyboard to use project conventions
- Use the dual footprints for futaba / cherry keys
- Include a diode for every key (dual SMT/TH options)
- Add stabilizers to the spacebar
- Add cherry and futaba aligner plates
- Add SMT resistor option
- Add unified retro keyboard text
Other:
- net class Default removed
- net class power1 removed
- net class signal removed
