File: hardware/keyboard-franklin-ace-1000/franklin-ace-1000-aligner-cherry/franklin-ace-1000-aligner-cherry.kicad_pcb (KiCad board)
At the start: 2 copper layers, 375.7 x 115.8 mm, 81 parts, among them K1 ESC, K10 A, K11 Z, K12 2 @, K13 W, K14 S, K15 X, K16 3 #, K17 E, K18 D, K19 C, K2 BREAK, K20 4 $, K21 R, K22 F, K23 V, K24 5 &, K25 T, K26 G, K27 B, K28 6 ^, K29 Y, K3 PAUSE, K30 H, K31 N, K32 SPACE_8U, K33 7 &, K34 U, K35 J, K36 M, K37 8 *, K38 I, K39 K, K4 CTRL, K40 , <, K41 9 (, K42 O, K43 L, K44 . >, K45 RIGHT, K46 -, K47 +, K48 *, K49 0 ), K5 TAB, K50 P, K51 ; :, K52 / ?, K53 7, K54 4, K55 1, K56 >, K57 - / _, K58 [ {, K59 ; ", K6 LOCK, K60 SHIFT, K61 8, K62 5, K63 2, K64 0, K65 + / =, K66 ] }, K67 RETURN, K68 LEFT, K69 9, K7 SHIFT, K70 6, K71 3, K72 ., K73 SPACE_1U, K74 TAB2, K9 Q

Commit message: More key fixes
Parts:
- added K8: 1 !, unikbd:Key_MX_Aligner, F.Cu at (164.1, 164.1)
- moved K66 7.14 mm to (390.3, 183.2)
- moved K58 2.38 mm to (366.5, 183.2)
Routing:
- net Row0: vias 0 -> 1
Other:
- board size 375.7 x 115.8 mm -> 383.5 x 113.5 mm
Changed lines of the file:
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@@
   (paper "A2")
   (title_block
-    (title "Franklin Ace Keyboard Cherry MX Aligner")
-    (date "2023-07-08")
+    (title "Franklin Ace 1000 keyboard cherry MX aligner")
+    (date "2023-10-01")
     (rev "1")
-    (company "Unifed Retro Keyboard Project")
-    (comment 1 "竜 クリストファー (Chris Ryu)}")
+    (company "Unified Retro Keyboard Project")
+    (comment 1 "竜 クリストファー (Chris Ryu) ")
     (comment 2 "Adapted by David Fenyes")
   )
@@
     )
     (pad_to_mask_clearance 0)
-    (grid_origin 121.412 199.6948)
     (pcbplotparams
       (layerselection 0x00010fc_ffffffff)
@@
   )
   (net 0 "")
+  (net 1 "Row0")
   (footprint "unikbd:Key_MX_Aligner" locked (layer "F.Cu")
     (at 282.998036 221.250352)
@@
   )
   (footprint "unikbd:Key_MX_Aligner" locked (layer "F.Cu")
-    (at 364.151036 183.150352)
+    (at 366.532286 183.150352)
     (property "Sheetfile" "franklin-ace-1000-keyboard.kicad_sch")
     (property "Sheetname" "")
@@
   )
   (footprint "unikbd:Key_MX_Aligner" locked (layer "F.Cu")
-    (at 383.201036 183.150352)
+    (at 390.344786 183.150352)
     (property "Sheetfile" "franklin-ace-1000-keyboard.kicad_sch")
     (property "Sheetname" "")
@@
   )
   (footprint "unikbd:Key_MX_Aligner" locked (layer "F.Cu")
+    (at 164.126036 164.100352)
+    (property "Sheetfile" "franklin-ace-1000-keyboard.kicad_sch")
+    (property "Sheetname" "")
+    (property "ki_description" "Generic connector, single row, 01x02, script generated")
+    (property "ki_keywords" "connector")
+    (attr through_hole)
+    (fp_text reference "K8" (at -5.0292 -7.7724) (layer "F.SilkS")
+        (effects (font (size 1 1) (thickness 0.15)))
+    )
+    (fp_text value "1 !" (at 0 7.9756) (layer "B.Fab")
+        (effects (font (size 1 1) (thickness 0.15)))
+    )
+    (fp_text user "${REFERENCE}" (at -2.54 -2.794) (layer "F.Fab")
+        (effects (font (size 1 1) (thickness 0.15)))
+    )
+    (fp_line (start -6.985 -6.8834) (end -6.985 7.0866)
+      (stroke (width 0.12) (type solid)) (layer "Edge.Cuts"))
+    (fp_line (start -6.985 -6.8834) (end 6.985 -6.8834)
+      (stroke (width 0.12) (type solid)) (layer "Edge.Cuts"))
+    (fp_line (start -6.985 7.0866) (end 6.985 7.0866)
+      (stroke (width 0.12) (type solid)) (layer "Edge.Cuts"))
+    (fp_line (start 6.985 7.0866) (end 6.985 -6.8834)
+      (stroke (width 0.12) (type solid)) (layer "Edge.Cuts"))
+  )
+  (footprint "unikbd:Key_MX_Aligner" locked (layer "F.Cu")
     (at 345.101036 183.150352)
     (property "Sheetfile" "franklin-ace-1000-keyboard.kicad_sch")
@@
       (stroke (width 0.12) (type solid)) (layer "Edge.Cuts"))
   )
-  (gr_line (start 110.5662 251.9) (end 486.3084 251.9)
+  (gr_line (start 491.49 138.43) (end 491.49 251.9)
     (stroke (width 0.1) (type solid)) (layer "Edge.Cuts"))
-  (gr_line (start 110.5662 251.9) (end 110.5662 136.0932)
+  (gr_line (start 107.95 251.9) (end 491.49 251.9)
     (stroke (width 0.1) (type solid)) (layer "Edge.Cuts"))
-  (gr_line (start 486.3084 136.0932) (end 110.5662 136.0932)
+  (gr_line (start 107.95 251.9) (end 107.95 138.43)
     (stroke (width 0.1) (type solid)) (layer "Edge.Cuts"))
-  (gr_line (start 486.3084 251.9) (end 486.3084 136.0932)
+  (gr_line (start 491.49 138.43) (end 107.95 138.43)
     (stroke (width 0.1) (type solid)) (layer "Edge.Cuts"))
-  (gr_text "${TITLE}\n${COMPANY}\nRev ${REVISION}   ${ISSUE_DATE}\n${COMMENT1}\n${COMMENT2}" (at 408.9908 241.1984) (layer "F.SilkS")
+  (gr_text "${TITLE}\n${COMPANY}\nRev ${REVISION}   ${ISSUE_DATE}\n${COMMENT1}\n${COMMENT2}" (at 400.05 241.3) (layer "F.SilkS")
     (effects (font (size 2 2) (thickness 0.3)) (justify left))
   )
+  (dimension (type aligned) (layer "Cmts.User")
+    (pts (xy 94.7 263.9) (xy 504.45 263.9))
+    (height 32.4)
+    (gr_text "16131.8898 mils" (at 299.575 295.15) (layer "Cmts.User")
+      (effects (font (size 1 1) (thickness 0.15)))
+    )
+    (format (prefix "") (suffix "") (units 3) (units_format 1) (precision 4))
+    (style (thickness 0.1) (arrow_length 1.27) (text_position_mode 0) (extension_height 0.58642) (extension_offset 0.5) keep_text_aligned)
+  )
+  (via (at 135.001 148.336) (size 0.8) (drill 0.4) (layers "F.Cu" "B.Cu") (net 1))
   (group "" (id e31c4550-33f7-4ba5-8b13-2f783de59f3a)
     (members
